File: 6bit-vga.kicad_pcb (KiCad board)
At the start: 2 copper layers, 40 x 40 mm, 150 parts, among them J1 pmod, J2 Conn_01x01, J3 Conn_01x01, J4 DB15_Female_HighDensity

Commit message: docs and kicad6 update
Other:
- net class Default removed
