File: 6bit-vga.kicad_pcb (KiCad board)
At the start: 2 copper layers, 40 x 40 mm, 150 parts, among them J1 pmod, J2 Conn_01x01, J3 Conn_01x01, J4 DB15_Female_HighDensity

Commit message: fixed bad fp
Parts:
- removed V10_14, V10_15, V10_6, V11_14, V13_14, V14_14, V16_14, V9_15, V9_6: AUTO_VIA, VIA_MATRIX
- added V10_17: AUTO_VIA, VIA_MATRIX, F.Cu at (120.4, 141.5)
- added V10_4: AUTO_VIA, VIA_MATRIX, F.Cu at (120.4, 108.5)
- added V11_13: AUTO_VIA, VIA_MATRIX, F.Cu at (122.9, 131.3)
- added V15_16: AUTO_VIA, VIA_MATRIX, F.Cu at (133.1, 138.9)
- added V16_16: AUTO_VIA, VIA_MATRIX, F.Cu at (135.6, 138.9)
- added V8_8: AUTO_VIA, VIA_MATRIX, F.Cu at (115.3, 118.6)
- added V9_17: AUTO_VIA, VIA_MATRIX, F.Cu at (117.9, 141.5)
- added V9_4: AUTO_VIA, VIA_MATRIX, F.Cu at (117.9, 108.5)

Commit message: update pcb and readme
Other:
- net class Default removed
